File: UINIO-USB-UART-CH343.kicad_pcb (KiCad board)
At the start: 2 copper layers, 33.7 x 20.3 mm, 25 parts, among them J4 Conn_01x03_Pin, J5 Conn_01x05_Pin, J6 Conn_01x04_Pin, J7 Conn_01x03_Pin, U2 CH343P

Commit message: Release UINIO-USB-UART-CH343 version 5.0.0.
Parts:
- moved C5 1.07 mm to (160.8, 98.3)
Routing:
- net /CH343_VDD_5V: track 35.7 -> 20.4 mm, vias 4 -> 5
- net GND: track 33.4 -> 41.8 mm, vias 35 -> 40
- net /CH343_USB_Data_P: track 13.9 -> 16.6 mm
- net Net-(D1-A): track 0.00 -> 1.35 mm
- net Net-(D5-K): track 0.39 -> 1.57 mm
- added copper zone on F.Cu, net /CH343_VDD_5V
